File: fluid sim pendant.kicad_sch (KiCad schematic)
At the start: 0 parts

Commit message: add parts to schematic
Parts:
- added USB1: TYPEC-304A-ACP16O, easyeda2kicad:USB-SMD_TYPEC-304A-ACP16O, symbol easyeda:TYPEC-304A-ACP16O
Changed lines of the file:
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@@
 	(generator_version "10.0")
 	(paper "A4")
+	(symbol
+		(lib_id "easyeda:TYPEC-304A-ACP16O")
+		(at 74.93 73.66 0)
+		(unit 1)
+		(body_style 1)
+		(exclude_from_sim no)
+		(in_bom yes)
+		(on_board yes)
+		(in_pos_files yes)
+		(dnp no)
+		(fields_autoplaced yes)
+		(property "Reference" "USB1"
+			(at 82.1533 59.69 0)
+			(show_name no)
+			(do_not_autoplace no)
+			(effects
+				(font
+					(size 1.27 1.27)
+				)
+				(justify left)
+			)
+		)
+		(property "Value" "TYPEC-304A-ACP16O"
+			(at 82.1533 62.23 0)
+			(show_name no)
+			(do_not_autoplace no)
+			(effects
+				(font
+					(size 1.27 1.27)
+				)
+				(justify left)
+			)
+		)
+		(property "Footprint" "easyeda2kicad:USB-SMD_TYPEC-304A-ACP16O"
+			(at 74.93 92.71 0)
+			(hide yes)
+			(show_name no)
+			(do_not_autoplace no)
+			(effects
+				(font
+					(size 1.27 1.27)
+				)
+			)
+		)
+		(property "Datasheet" "https://www.lcsc.com/datasheet/C2909610.pdf"
+			(at 74.93 95.25 0)
+			(hide yes)
+			(show_name no)
+			(do_not_autoplace no)
+			(effects
+				(font
+					(size 1.27 1.27)
+				)
+			)
+		)
+		(property "Description" ""
+			(at 74.93 73.66 0)
+			(hide yes)
+			(show_name no)
+			(do_not_autoplace no)
+			(effects
+				(font
+					(size 1.27 1.27)
+				)
+			)
+		)
+		(property "Manufacturer" "XUNPU(讯普)"
+			(at 74.93 97.79 0)
+			(hide yes)
+			(show_name no)
+			(do_not_autoplace no)
+			(effects
+				(font
+					(size 1.27 1.27)
+				)
+			)
+		)
+		(property "MPN" "TYPEC-304A-ACP16O"
+			(at 74.93 100.33 0)
+			(hide yes)
+			(show_name no)
+			(do_not_autoplace no)
+			(effects
+				(font
+					(size 1.27 1.27)
+				)
+			)
+		)
+		(property "LCSC Part" "C2909610"
+			(at 74.93 102.87 0)
+			(hide yes)
+			(show_name no)
+			(do_not_autoplace no)
+			(effects
+				(font
+					(size 1.27 1.27)
+				)
+			)
+		)
+		(pin "B7"
+		)
+		(pin "A7"
+		)
+		(pin "15"
+		)
+		(pin "A1B12"
+		)
+		(pin "A6"
+		)
+		(pin "A5"
+		)
+		(pin "14"
+		)
+		(pin "A4B9"
+		)
+		(pin "B1A12"
+		)
+		(pin "B4A9"
+		)
+		(pin "12"
+		)
+		(pin "B5"
+		)
+		(pin "B6"
+		)
+		(pin "13"
+		)
+		(pin "A8"
+		)
+		(pin "B8"
+		)
+		(instances
+			(project "fluid sim pendant"
+				(path "/db935d3a-e302-4204-8da6-cdf8740661d6"
+					(reference "USB1")
+					(unit 1)
+				)
+			)
+		)
+	)
 	(sheet_instances
 		(path "/"
